Commit message: Add files via upload

File: urdf/hand.urdf (robot description, URDF)
Before this commit: robot hand, 14 links, 13 joints
Links:
- removed link wrist
- added link palm-base, mass 1.0; collision cylinder length=0.5 radius=1.75; visual cylinder length=0.5 radius=1.75
- added link stand, mass 1000; collision cylinder length=0.5 radius=1.5; visual cylinder length=0.5 radius=1.5
- link palm: geometry collision box size=3.5 2 0.5; visual box size=3.5 2 0.51
Joints:
- removed joint palm-wrist
- added joint palm: type fixed, parent palm-base, child palm, origin xyz=0 0 0 rpy=0 0 0
- added joint stand: type fixed, parent stand, child palm-base, origin xyz=0 0 0 rpy=0 0 0
